Commit message: 4/1/2026 thong luong

File: src/my_sr_arm_rb/urdf/my_sr_arm_rb.urdf (robot description, URDF)
Before this commit: robot my_sr_arm_rb, 21 links, 20 joints
Links:
- removed link base_footprint
- added link world
- link banh_phai: mass 0.11437626123491 -> 0.114; geometry collision mesh filename=file:///home/nguyen1/ros2_rnea_control/src/my_sr_arm_rb/mes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; visual mesh filename=file:///home/nguyen1/ros2_rnea_control/src/my_sr_arm_rb/mes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
- link banh_phu_1: geometry collision mesh filename=file:///home/nguyen1/ros2_rnea_control/src/my_sr_arm_rb/mes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; visual mesh filename=file:///home/nguyen1/ros2_rnea_control/src/my_sr_arm_rb/mes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
- link banh_phu_2: mass 0.00669807920710659 -> 0.00669; geometry collision mesh filename=file:///home/nguyen1/ros2_rnea_control/src/my_sr_arm_rb/mes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; visual mesh filename=file:///home/nguyen1/ros2_rnea_control/src/my_sr_arm_rb/mes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
- link banh_trai: mass 0.11437626123491 -> 0.114; geometry collision mesh filename=file:///home/nguyen1/ros2_rnea_control/src/my_sr_arm_rb/mes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; visual mesh filename=file:///home/nguyen1/ros2_rnea_control/src/my_sr_arm_rb/mes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
- link base_link: geometry collision mesh filename=file:///home/nguyen1/ros2_rnea_control/src/my_sr_arm_rb/mes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; visual mesh filename=file:///home/nguyen1/ros2_rnea_control/src/my_sr_arm_rb/mes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
- link link_1: geometry collision mesh filename=file:///home/nguyen1/ros2_rnea_control/src/my_sr_arm_rb/mes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; visual mesh filename=file:///home/nguyen1/ros2_rnea_control/src/my_sr_arm_rb/mes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
- link link_2: geometry collision mesh filename=file:///home/nguyen1/ros2_rnea_control/src/my_sr_arm_rb/mes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; visual mesh filename=file:///home/nguyen1/ros2_rnea_control/src/my_sr_arm_rb/mes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
- link link_3: geometry collision mesh filename=file:///home/nguyen1/ros2_rnea_control/src/my_sr_arm_rb/mes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; visual mesh filename=file:///home/nguyen1/ros2_rnea_control/src/my_sr_arm_rb/mes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
- link link_4: geometry collision mesh filename=file:///home/nguyen1/ros2_rnea_control/src/my_sr_arm_rb/mes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; visual mesh filename=file:///home/nguyen1/ros2_rnea_control/src/my_sr_arm_rb/mes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
- link link_5: geometry collision mesh filename=file:///home/nguyen1/ros2_rnea_control/src/my_sr_arm_rb/mes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; visual mesh filename=file:///home/nguyen1/ros2_rnea_control/src/my_sr_arm_rb/mes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
- link link_sr_11: mass 0.0643607669234624 -> 0.06; geometry visual mesh filename=file:///home/nguyen1/ros2_rnea_control/src/my_sr_arm_rb/mes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
- link link_sr_12: mass 0.0643607669234623 -> 0.06; geometry visual mesh filename=file:///home/nguyen1/ros2_rnea_control/src/my_sr_arm_rb/mes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
- link link_sr_13: mass 0.0643607669234624 -> 0.06; geometry collision mesh filename=file:///home/nguyen1/ros2_rnea_control/src/my_sr_arm_rb/mes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; visual mesh filename=file:///home/nguyen1/ros2_rnea_control/src/my_sr_arm_rb/mes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
- link link_sr_14: mass 0.0643607669234623 -> 0.06; geometry collision mesh filename=file:///home/nguyen1/ros2_rnea_control/src/my_sr_arm_rb/mes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; visual mesh filename=file:///home/nguyen1/ros2_rnea_control/src/my_sr_arm_rb/mes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
- link link_sr_21: mass 0.0824501328250599 -> 0.08; geometry visual mesh filename=file:///home/nguyen1/ros2_rnea_control/src/my_sr_arm_rb/mes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
- link link_sr_22: mass 0.0824501328250598 -> 0.08; geometry visual mesh filename=file:///home/nguyen1/ros2_rnea_control/src/my_sr_arm_rb/mes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
- link link_sr_23: mass 0.0824501328250598 -> 0.08; geometry collision mesh filename=file:///home/nguyen1/ros2_rnea_control/src/my_sr_arm_rb/mes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; visual mesh filename=file:///home/nguyen1/ros2_rnea_control/src/my_sr_arm_rb/mes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
- link link_sr_24: mass 0.0824501328250598 -> 0.08; geometry visual mesh filename=file:///home/nguyen1/ros2_rnea_control/src/my_sr_arm_rb/mes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
Joints:
- removed joint base_footprint_to_base_link_joint
- added joint world_to_base_link_joint: type fixed, parent world, child base_link, origin xyz=0 0 0 rpy=0 0 1.5708
- joint joint_sr_14: origin xyz=-0.109999999999999 -0.135000000000001 0.1175 rpy=-1.5707963267949 0 -3.14159265358979 -> xyz=-0.11 -0.135 0.1175 rpy=-1.5708 0 -3.14159

File: src/my_sr_arm_rb/urdf/test.urdf (robot description, URDF)
Before this commit: robot sr_arm_robot, 2 links, 1 joints
Links:
- removed link link1
- added link banh_phai, mass 0.11437626123491; collision mesh filename=file:///home/nguyen1/ros2_rnea_control/src/my_sr_arm_rb/mes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; visual mesh filename=file:///home/nguyen1/ros2_rnea_control/src/my_sr_arm_rb/mes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
- added link banh_phu_1, mass 0.00541003378791435; collision mesh filename=file:///home/nguyen1/ros2_rnea_control/src/my_sr_arm_rb/mes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; visual mesh filename=file:///home/nguyen1/ros2_rnea_control/src/my_sr_arm_rb/mes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
- added link banh_phu_2, mass 0.00669807920710659; collision mesh filename=file:///home/nguyen1/ros2_rnea_control/src/my_sr_arm_rb/mes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; visual mesh filename=file:///home/nguyen1/ros2_rnea_control/src/my_sr_arm_rb/mes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
- added link banh_trai, mass 0.11437626123491; collision mesh filename=file:///home/nguyen1/ros2_rnea_control/src/my_sr_arm_rb/mes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; visual mesh filename=file:///home/nguyen1/ros2_rnea_control/src/my_sr_arm_rb/mes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
- added link base_footprint
- added link gripper, mass 1e-5; visual sphere radius=0.001
- added link laser_link, mass 1e-5; collision box size=0.1 0.1 0.1; visual cylinder length=0.07 radius=0.04
- added link link_1, mass 0.83811; collision mesh filename=file:///home/nguyen1/ros2_rnea_control/src/my_sr_arm_rb/mes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; visual mesh filename=file:///home/nguyen1/ros2_rnea_control/src/my_sr_arm_rb/mes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
- added link link_2, mass 0.28679331350207; collision mesh filename=file:///home/nguyen1/ros2_rnea_control/src/my_sr_arm_rb/mes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; visual mesh filename=file:///home/nguyen1/ros2_rnea_control/src/my_sr_arm_rb/mes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
- added link link_3, mass 0.497898478741613; collision mesh filename=file:///home/nguyen1/ros2_rnea_control/src/my_sr_arm_rb/mes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; visual mesh filename=file:///home/nguyen1/ros2_rnea_control/src/my_sr_arm_rb/mes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
- added link link_4, mass 0.427287350838624; collision mesh filename=file:///home/nguyen1/ros2_rnea_control/src/my_sr_arm_rb/mes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; visual mesh filename=file:///home/nguyen1/ros2_rnea_control/src/my_sr_arm_rb/mes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
- added link link_5, mass 0.0474207074268081; collision mesh filename=file:///home/nguyen1/ros2_rnea_control/src/my_sr_arm_rb/mes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; visual mesh filename=file:///home/nguyen1/ros2_rnea_control/src/my_sr_arm_rb/mes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
- added link link_sr_11, mass 0.0643607669234624; collision mesh filename=file:///home/nguyen1/ros2_rnea_control/src/my_sr_arm_rb/mes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; visual mesh filename=file:///home/nguyen1/ros2_rnea_control/src/my_sr_arm_rb/mes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
- added link link_sr_12, mass 0.0643607669234623; collision mesh filename=file:///home/nguyen1/ros2_rnea_control/src/my_sr_arm_rb/mes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; visual mesh filename=file:///home/nguyen1/ros2_rnea_control/src/my_sr_arm_rb/mes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
- added link link_sr_13, mass 0.0643607669234624; collision mesh filename=file:///home/nguyen1/ros2_rnea_control/src/my_sr_arm_rb/mes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; visual mesh filename=file:///home/nguyen1/ros2_rnea_control/src/my_sr_arm_rb/mes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
- added link link_sr_14, mass 0.0643607669234623; collision mesh filename=file:///home/nguyen1/ros2_rnea_control/src/my_sr_arm_rb/mes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; visual mesh filename=file:///home/nguyen1/ros2_rnea_control/src/my_sr_arm_rb/mes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
- added link link_sr_21, mass 0.0824501328250599; collision mesh filename=file:///home/nguyen1/ros2_rnea_control/src/my_sr_arm_rb/mes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; visual mesh filename=file:///home/nguyen1/ros2_rnea_control/src/my_sr_arm_rb/mes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
- added link link_sr_22, mass 0.0824501328250598; collision mesh filename=file:///home/nguyen1/ros2_rnea_control/src/my_sr_arm_rb/mes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; visual mesh filename=file:///home/nguyen1/ros2_rnea_control/src/my_sr_arm_rb/mes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
- added link link_sr_23, mass 0.0824501328250598; collision mesh filename=file:///home/nguyen1/ros2_rnea_control/src/my_sr_arm_rb/mes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; visual mesh filename=file:///home/nguyen1/ros2_rnea_control/src/my_sr_arm_rb/mes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
- added link link_sr_24, mass 0.0824501328250598; collision mesh filename=file:///home/nguyen1/ros2_rnea_control/src/my_sr_arm_rb/mes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; visual mesh filename=file:///home/nguyen1/ros2_rnea_control/src/my_sr_arm_rb/mes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
- link base_link: mass 1.0 -> 9.51282461066678; geometry collision mesh filename=file:///home/nguyen1/ros2_rnea_control/src/my_sr_arm_rb/mes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; visual mesh filename=file:///home/nguyen1/ros2_rnea_control/src/my_sr_arm_rb/mes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
Joints:
- removed joint joint1
- added joint base_footprint_to_base_link_joint: type fixed, parent base_footprint, child base_link, origin xyz=0 0 0 rpy=0 0 1.5708
- added joint joint_1: type prismatic, parent base_link, child link_1, origin xyz=0 0 0.1175 rpy=0 0 0, axis 0 0 1, limit lower=0 upper=0.25 effort=100 velocity=10
- added joint joint_2: type revolute, parent link_1, child link_2, origin xyz=0 0 0.0705288076205608 rpy=0 0 0, axis 0 0 1, limit lower=-3.14 upper=3.14 effort=10 velocity=10
- added joint joint_3: type revolute, parent link_2, child link_3, origin xyz=0 0 0.05 rpy=1.5708 0 -1.5708, axis 0 0 1, limit lower=0 upper=3.14 effort=10 velocity=10
- added joint joint_4: type revolute, parent link_3, child link_4, origin xyz=0.20006 -0.00084852 0.0012303 rpy=0 0 0, axis 0 0 1, limit lower=-1.57 upper=1.57 effort=10 velocity=10
- added joint joint_5: type revolute, parent link_4, child link_5, origin xyz=0.14999 -0.00132 0.00092242 rpy=0 -0.0061498 0, axis 0 0 1, limit lower=-1.57 upper=1.57 effort=10 velocity=10
- added joint joint_banh_phai: type continuous, parent base_link, child banh_phai, origin xyz=-0.17 0.125 0.0405 rpy=1.5708 0 1.5708, axis 0 0 1
- added joint joint_banh_trai: type continuous, parent base_link, child banh_trai, origin xyz=0.17 0.125 0.0405 rpy=-1.5708 0 -1.5708, axis 0 0 1
- added joint joint_bp_1: type continuous, parent base_link, child banh_phu_1, origin xyz=0 -0.1822 0.03 rpy=0 0 -1.0422, axis 0 0 1
- added joint joint_bp_2: type continuous, parent banh_phu_1, child banh_phu_2, origin xyz=0.012473 0.014786 -0.015 rpy=-1.5708 0 0, axis 0 0 1
- added joint joint_gripper: type fixed, parent link_5, child gripper, origin xyz=0.05 0 0 rpy=0 0 0
- added joint joint_sr_11: type revolute, parent base_link, child link_sr_11, origin xyz=0.135 -0.11 0.1175 rpy=-1.5708 0 -1.5708, axis 0 0 1, limit lower=-0.785 upper=0.785 effort=10 velocity=10
- added joint joint_sr_12: type revolute, parent base_link, child link_sr_12, origin xyz=0.11 0.135 0.1175 rpy=-1.5708 0 0, axis 0 0 1, limit lower=-0.758 upper=0.758 effort=10 velocity=10
- added joint joint_sr_13: type revolute, parent base_link, child link_sr_13, origin xyz=-0.135 0.11 0.1175 rpy=-1.5708 0 1.5708, axis 0 0 1, limit lower=-0.785 upper=0.785 effort=10 velocity=10
- added joint joint_sr_14: type continuous, parent base_link, child link_sr_14, origin xyz=-0.109999999999999 -0.135000000000001 0.1175 rpy=-1.5707963267949 0 -3.14159265358979, axis 0 0 1, limit lower=-0.785 upper=0.785 effort=10 velocity=10
- added joint joint_sr_21: type revolute, parent link_sr_11, child link_sr_21, origin xyz=-0.12582 -0.098839 0 rpy=0 0 -2.4757, axis 0 0 1, limit lower=-3.14 upper=3.14 effort=10 velocity=10
- added joint joint_sr_22: type revolute, parent link_sr_12, child link_sr_22, origin xyz=-0.12582 -0.098839 0 rpy=0 0 -2.4757, axis 0 0 1, limit lower=-3.14 upper=3.14 effort=10 velocity=10
- added joint joint_sr_23: type revolute, parent link_sr_13, child link_sr_23, origin xyz=-0.12582 -0.098839 0 rpy=0 0 -2.4757, axis 0 0 1, limit lower=-3.14 upper=3.14 effort=10 velocity=10
- added joint joint_sr_24: type revolute, parent link_sr_14, child link_sr_24, origin xyz=-0.12582 -0.098839 0 rpy=0 0 -2.4757, axis 0 0 1, limit lower=-3.14 upper=3.14 effort=10 velocity=10
- added joint laser_joint: type fixed, parent base_link, child laser_link, origin xyz=0 0 0.15 rpy=0 0 0

Commit message: trajectory ee fl

File: src/my_sr_arm_rb/urdf/my_sr_arm_rb.urdf (robot description, URDF)
Before this commit: robot my_sr_arm_rb, 21 links, 20 joints
Links:
- removed link gripper
- added link gripper1, mass 0.00889698927943615; collision mesh filename=file:///home/nguyen1/ros2_rnea_control/src/my_sr_arm_rb/mes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; visual mesh filename=file:///home/nguyen1/ros2_rnea_control/src/my_sr_arm_rb/mes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
- added link gripper2, mass 0.00889698927943615; collision mesh filename=file:///home/nguyen1/ros2_rnea_control/src/my_sr_arm_rb/mes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; visual mesh filename=file:///home/nguyen1/ros2_rnea_control/src/my_sr_arm_rb/mes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
Joints:
- removed joint joint_gripper
- added joint joint_gripper1: type prismatic, parent link_5, child gripper1, origin xyz=0.093041 -2.978E-05 0.00068173 rpy=0.043655 0 0, axis 0 0 -1, limit lower=-0.02 upper=0 effort=0 velocity=0
- added joint joint_gripper2: type prismatic, parent link_5, child gripper2, origin xyz=0.093041 -1.3971E-05 0.00031983 rpy=-3.0979 0 0, axis 0 0 1, limit lower=0 upper=0.02 effort=0 velocity=0

File: src/my_sr_arm_rb/urdf/test.urdf (robot description, URDF)
Before this commit: robot my_sr_arm_rb, 21 links, 20 joints
Links:
- removed link banh_phai
- removed link banh_phu_1
- removed link banh_phu_2
- removed link banh_trai
- removed link base_footprint
- removed link gripper
- removed link laser_link
- removed link link_sr_11
- removed link link_sr_12
- removed link link_sr_13
- removed link link_sr_14
- removed link link_sr_21
- removed link link_sr_22
- removed link link_sr_23
- removed link link_sr_24
- added link ga, mass 0.00691409738978907; collision mesh filename=file:///home/nguyen1/ros2_rnea_control/src/my_sr_arm_rb/mes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; visual mesh filename=file:///home/nguyen1/ros2_rnea_control/src/my_sr_arm_rb/mes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
- added link gripper1, mass 0.00889698927943615; collision mesh filename=file:///home/nguyen1/ros2_rnea_control/src/my_sr_arm_rb/mes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; visual mesh filename=file:///home/nguyen1/ros2_rnea_control/src/my_sr_arm_rb/mes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
- added link gripper2, mass 0.00889698927943615; collision mesh filename=file:///home/nguyen1/ros2_rnea_control/src/my_sr_arm_rb/mes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; visual mesh filename=file:///home/nguyen1/ros2_rnea_control/src/my_sr_arm_rb/mes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
- added link link_sr11, mass 0.0987537674712606; collision mesh filename=file:///home/nguyen1/ros2_rnea_control/src/my_sr_arm_rb/mes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; visual mesh filename=file:///home/nguyen1/ros2_rnea_control/src/my_sr_arm_rb/mes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
- added link link_sr12, mass 0.0987537674712605; collision mesh filename=file:///home/nguyen1/ros2_rnea_control/src/my_sr_arm_rb/mes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; visual mesh filename=file:///home/nguyen1/ros2_rnea_control/src/my_sr_arm_rb/mes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
- added link link_sr13, mass 0.0987537674712604; collision mesh filename=file:///home/nguyen1/ros2_rnea_control/src/my_sr_arm_rb/mes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; visual mesh filename=file:///home/nguyen1/ros2_rnea_control/src/my_sr_arm_rb/mes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
- added link link_sr14, mass 0.0987537674712606; collision mesh filename=file:///home/nguyen1/ros2_rnea_control/src/my_sr_arm_rb/mes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; visual mesh filename=file:///home/nguyen1/ros2_rnea_control/src/my_sr_arm_rb/mes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
- added link link_sr21, mass 0.10234077696469; collision mesh filename=file:///home/nguyen1/ros2_rnea_control/src/my_sr_arm_rb/mes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; visual mesh filename=file:///home/nguyen1/ros2_rnea_control/src/my_sr_arm_rb/mes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
- added link link_sr22, mass 0.10234077696469; collision mesh filename=file:///home/nguyen1/ros2_rnea_control/src/my_sr_arm_rb/mes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; visual mesh filename=file:///home/nguyen1/ros2_rnea_control/src/my_sr_arm_rb/mes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
- added link link_sr23, mass 0.102340776964689; collision mesh filename=file:///home/nguyen1/ros2_rnea_control/src/my_sr_arm_rb/mes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; visual mesh filename=file:///home/nguyen1/ros2_rnea_control/src/my_sr_arm_rb/mes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
- added link link_sr24, mass 0.10234077696469; collision mesh filename=file:///home/nguyen1/ros2_rnea_control/src/my_sr_arm_rb/mes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; visual mesh filename=file:///home/nguyen1/ros2_rnea_control/src/my_sr_arm_rb/mes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
- added link wheel_3, mass 0.00795501647667156; collision mesh filename=file:///home/nguyen1/ros2_rnea_control/src/my_sr_arm_rb/mes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; visual mesh filename=file:///home/nguyen1/ros2_rnea_control/src/my_sr_arm_rb/mes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
- added link wheel_L, mass 0.11437626123491; collision mesh filename=file:///home/nguyen1/ros2_rnea_control/src/my_sr_arm_rb/mes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; visual mesh filename=file:///home/nguyen1/ros2_rnea_control/src/my_sr_arm_rb/mes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
- added link wheel_R, mass 0.11437626123491; collision mesh filename=file:///home/nguyen1/ros2_rnea_control/src/my_sr_arm_rb/mes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; visual mesh filename=file:///home/nguyen1/ros2_rnea_control/src/my_sr_arm_rb/mes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
- added link world
- link base_link: mass 9.51282461066678 -> 9.43905709432116
- link link_1: mass 0.83811 -> 0.784333797437522
- link link_4: mass 0.427287350838624 -> 0.427287364630589
- link link_5: mass 0.0474207074268081 -> 0.0592833623022146
Joints:
- removed joint base_footprint_to_base_link_joint
- removed joint joint_banh_phai
- removed joint joint_banh_trai
- removed joint joint_bp_1
- removed joint joint_bp_2
- removed joint joint_gripper
- removed joint joint_sr_11
- removed joint joint_sr_12
- removed joint joint_sr_13
- removed joint joint_sr_14
- removed joint joint_sr_21
- removed joint joint_sr_22
- removed joint joint_sr_23
- removed joint joint_sr_24
- removed joint laser_joint
- added joint joint_ga: type revolute, parent base_link, child ga, origin xyz=0.182204093751995 0 0 rpy=0 0 0, axis 0 0 -1, limit lower=0 upper=0 effort=0 velocity=0
- added joint joint_gripper1: type prismatic, parent link_5, child gripper1, origin xyz=0.093041 -2.978E-05 0.00068173 rpy=0.043655 0 0, axis 0 0 -1, limit lower=-0.1 upper=0 effort=0 velocity=0
- added joint joint_gripper2: type prismatic, parent link_5, child gripper2, origin xyz=0.093041 -1.3971E-05 0.00031983 rpy=-3.0979 0 0, axis 0 0 1, limit lower=0 upper=0.1 effort=0 velocity=0
- added joint joint_sr11: type revolute, parent base_link, child link_sr11, origin xyz=-0.109999999999998 -0.132000000000001 0.0775 rpy=1.5707963267949 0 0, axis 0 0 1, limit lower=0.3 upper=1.5 effort=0 velocity=0
- added joint joint_sr12: type revolute, parent base_link, child link_sr12, origin xyz=0.132000000000001 -0.109999999999999 0.0775 rpy=1.5707963267949 0 1.5707963267949, axis 0 0 1, limit lower=0.3 upper=1.5 effort=0 velocity=0
- added joint joint_sr13: type revolute, parent base_link, child link_sr13, origin xyz=0.109999999999999 0.132000000000001 0.0775 rpy=1.5707963267949 0 -3.14159265358979, axis 0 0 1, limit lower=0.3 upper=1.5 effort=0 velocity=0
- added joint joint_sr14: type revolute, parent base_link, child link_sr14, origin xyz=-0.132000000000001 0.109999999999999 0.0775 rpy=1.5707963267949 0 -1.57079632679489, axis 0 0 1, limit lower=0.3 upper=1.5 effort=0 velocity=0
- added joint joint_sr21: type revolute, parent link_sr11, child link_sr21, origin xyz=0.222051464893497 0.012089124809175 0.00299999999999787 rpy=0 0 -0.00410256010962525, axis 0 0 1, limit lower=0 upper=0 effort=0 velocity=0
- added joint joint_sr22: type revolute, parent link_sr12, child link_sr22, origin xyz=0.222051464893497 0.0120891248091607 0.00300000000000081 rpy=0 0 -0.00410256010968941, axis 0 0 1, limit lower=0.3 upper=1.5 effort=0 velocity=0
- added joint joint_sr23: type revolute, parent link_sr13, child link_sr23, origin xyz=0.222051464893498 0.0120891248091449 0.00300000000000061 rpy=0 0 -0.00410256010976083, axis 0 0 1, limit lower=0.3 upper=1.5 effort=0 velocity=0
- added joint joint_sr24: type revolute, parent link_sr14, child link_sr24, origin xyz=0.222051464893499 0.012089124809125 0.00300000000000075 rpy=0 0 0, axis 0 0 1, limit lower=0.3 upper=1.5 effort=0 velocity=0
- added joint joint_wheel3: type revolute, parent ga, child wheel_3, origin xyz=0.012385518488979 -0.00149025686129269 -0.0249996271077275 rpy=-1.5707963267949 0 -0.102617805790671, axis 0 0 -1, limit lower=0 upper=0 effort=0 velocity=0
- added joint joint_wheel_L: type revolute, parent base_link, child wheel_L, origin xyz=-0.125 0.16 0.000499999999999995 rpy=-1.5707963267949 0 0, axis 0 0 1, limit lower=0 upper=0 effort=0 velocity=0
- added joint joint_wheel_R: type revolute, parent base_link, child wheel_R, origin xyz=-0.125 -0.16 0.000499999999999992 rpy=1.5707963267949 0 0, axis 0 0 -1, limit lower=0 upper=0 effort=0 velocity=0
- added joint world_joint: type fixed, parent world, child base_link, origin xyz=0 0 0.05 rpy=0 0 0
- joint joint_1: limit lower=0 upper=0.25 effort=100 velocity=10 -> lower=0 upper=0.44 effort=0 velocity=0; origin xyz=0 0 0.1175 rpy=0 0 0 -> xyz=0 0 0.106678249618277 rpy=0 0 0
- joint joint_2: limit lower=-3.14 upper=3.14 effort=10 velocity=10 -> lower=-3.14 upper=3.14 effort=0 velocity=0; origin xyz=0 0 0.0705288076205608 rpy=0 0 0 -> xyz=0 0 0 rpy=0 0 0.000962225911754787
- joint joint_3: axis 0 0 1 -> -0.00096222576328123 0 -0.999999537060683; limit lower=0 upper=3.14 effort=10 velocity=10 -> lower=0 upper=3.14 effort=0 velocity=0; origin xyz=0 0 0.05 rpy=1.5708 0 -1.5708 -> xyz=0 0 0.05 rpy=1.5707963267949 0 -0.000962225911765263
- joint joint_4: axis 0 0 1 -> 0 -0.291324505694131 0.956624290085753; limit lower=-1.57 upper=1.57 effort=10 velocity=10 -> lower=-1.57 upper=1.57 effort=0 velocity=0; origin xyz=0.20006 -0.00084852 0.0012303 rpy=0 0 0 -> xyz=0.200048866595845 0.00266483542377308 -0.0001924922624659 rpy=-0.295608068156452 0.000962221108556715 0.00315967556313662
- joint joint_5: axis 0 0 1 -> 0 -0.0436412506776905 0.999047266769339; limit lower=-1.57 upper=1.57 effort=10 velocity=10 -> lower=-1.57 upper=1.57 effort=0 velocity=0; origin xyz=0.14999 -0.00132 0.00092242 rpy=0 -0.0061498 0 -> xyz=0.15 0 0 rpy=0.251906378391343 -0.00549689269092315 0.0180513465975973
