Commit message: chia module

File: src/my_sr_arm_rb/urdf/my_sr_arm_rb.urdf (robot description, URDF)
Before this commit: robot my_sr_arm_rb, 22 links, 21 joints
Links:
- link banh_phai: geometry collision mesh filename=file:///home/nguyen1/workspace/ros2_rnea_control/src/my_sr_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; visual mesh filename=file:///home/nguyen1/workspace/ros2_rnea_control/src/my_sr_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
- link banh_phu_1: geometry collision mesh filename=file:///home/nguyen1/workspace/ros2_rnea_control/src/my_sr_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; visual mesh filename=file:///home/nguyen1/workspace/ros2_rnea_control/src/my_sr_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
- link banh_phu_2: geometry collision mesh filename=file:///home/nguyen1/workspace/ros2_rnea_control/src/my_sr_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; visual mesh filename=file:///home/nguyen1/workspace/ros2_rnea_control/src/my_sr_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
- link banh_trai: geometry collision mesh filename=file:///home/nguyen1/workspace/ros2_rnea_control/src/my_sr_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; visual mesh filename=file:///home/nguyen1/workspace/ros2_rnea_control/src/my_sr_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
- link base_link: geometry collision mesh filename=file:///home/nguyen1/workspace/ros2_rnea_control/src/my_sr_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; visual mesh filename=file:///home/nguyen1/workspace/ros2_rnea_control/src/my_sr_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
- link gripper1: geometry collision mesh filename=file:///home/nguyen1/workspace/ros2_rnea_control/src/my_sr_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; visual mesh filename=file:///home/nguyen1/workspace/ros2_rnea_control/src/my_sr_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
- link gripper2: geometry collision mesh filename=file:///home/nguyen1/workspace/ros2_rnea_control/src/my_sr_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; visual mesh filename=file:///home/nguyen1/workspace/ros2_rnea_control/src/my_sr_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
- link link_1: geometry collision mesh filename=file:///home/nguyen1/workspace/ros2_rnea_control/src/my_sr_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; visual mesh filename=file:///home/nguyen1/workspace/ros2_rnea_control/src/my_sr_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
- link link_2: geometry collision mesh filename=file:///home/nguyen1/workspace/ros2_rnea_control/src/my_sr_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; visual mesh filename=file:///home/nguyen1/workspace/ros2_rnea_control/src/my_sr_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
- link link_3: geometry collision mesh filename=file:///home/nguyen1/workspace/ros2_rnea_control/src/my_sr_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; visual mesh filename=file:///home/nguyen1/workspace/ros2_rnea_control/src/my_sr_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
- link link_4: geometry collision mesh filename=file:///home/nguyen1/workspace/ros2_rnea_control/src/my_sr_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; visual mesh filename=file:///home/nguyen1/workspace/ros2_rnea_control/src/my_sr_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
- link link_5: geometry collision mesh filename=file:///home/nguyen1/workspace/ros2_rnea_control/src/my_sr_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; visual mesh filename=file:///home/nguyen1/workspace/ros2_rnea_control/src/my_sr_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
- link link_sr_11: geometry visual mesh filename=file:///home/nguyen1/workspace/ros2_rnea_control/src/my_sr_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
- link link_sr_12: geometry visual mesh filename=file:///home/nguyen1/workspace/ros2_rnea_control/src/my_sr_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
- link link_sr_13: geometry collision mesh filename=file:///home/nguyen1/workspace/ros2_rnea_control/src/my_sr_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; visual mesh filename=file:///home/nguyen1/workspace/ros2_rnea_control/src/my_sr_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
- link link_sr_14: geometry collision mesh filename=file:///home/nguyen1/workspace/ros2_rnea_control/src/my_sr_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; visual mesh filename=file:///home/nguyen1/workspace/ros2_rnea_control/src/my_sr_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
- link link_sr_21: geometry visual mesh filename=file:///home/nguyen1/workspace/ros2_rnea_control/src/my_sr_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
- link link_sr_22: geometry visual mesh filename=file:///home/nguyen1/workspace/ros2_rnea_control/src/my_sr_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
- link link_sr_23: geometry collision mesh filename=file:///home/nguyen1/workspace/ros2_rnea_control/src/my_sr_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; visual mesh filename=file:///home/nguyen1/workspace/ros2_rnea_control/src/my_sr_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
- link link_sr_24: geometry visual mesh filename=file:///home/nguyen1/workspace/ros2_rnea_control/src/my_sr_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
